Commit message: urdfs have tf_prefix

File: base_urdf2_description/urdf/base_urdf2.xacro (robot description, xacro)
@@ -5,5 +5,5 @@
 <xacro:include filename="$(find base_urdf2_description)/urdf/base_urdf2.gazebo" />
 <xacro:arg name="tf_prefix" default=""/>
-<link name="$(arg tf_prefix)base_link">
+<link name="$(arg tf_prefix)/base_link">
   <inertial>
     <origin rpy="0 0 0" xyz="0.030118479856442667 5.481613643184651e-07 0.01884821678256087"/>
@@ -171,5 +171,5 @@
   </collision>
 </link>
-<link name="$(arg tf_prefix)Wheel_Assy_01_1">
+<link name="$(arg tf_prefix)/Wheel_Assy_01_1">
   <inertial>
     <origin rpy="0 0 0" xyz="1.5818095039366042e-07 -0.054036798760615096 -8.681375665453572e-05"/>
@@ -211,5 +211,5 @@
   </collision>
 </link>
-<link name="$(arg tf_prefix)Wheel_Assy_01_2">
+<link name="$(arg tf_prefix)/Wheel_Assy_01_2">
   <inertial>
     <origin rpy="0 0 0" xyz="1.5818095050468273e-07 0.3740367987606148 8.681375665499716e-05"/>
@@ -253,12 +253,12 @@
 <joint name="Rev9" type="continuous">
   <origin rpy="0 0 0" xyz="0.21011 -0.16 -0.03"/>
-  <parent link="$(arg tf_prefix)base_link"/>
-  <child link="$(arg tf_prefix)Wheel_Assy_01_1"/>
+  <parent link="$(arg tf_prefix)/base_link"/>
+  <child link="$(arg tf_prefix)/Wheel_Assy_01_1"/>
   <axis xyz="-0.0 -1.0 -0.0"/>
 </joint>
 <joint name="Rev10" type="continuous">
   <origin rpy="0 0 0" xyz="0.21011 -0.16 -0.03"/>
-  <parent link="$(arg tf_prefix)base_link"/>
-  <child link="$(arg tf_prefix)Wheel_Assy_01_2"/>
+  <parent link="$(arg tf_prefix)/base_link"/>
+  <child link="$(arg tf_prefix)/Wheel_Assy_01_2"/>
   <axis xyz="-0.0 -1.0 -0.0"/>
 </joint>

File: grip_urdf1_description/urdf/grip_urdf1.xacro (robot description, xacro)
@@ -5,5 +5,5 @@
 <xacro:include filename="$(find grip_urdf1_description)/urdf/grip_urdf1.gazebo" />
 <xacro:arg name="tf_prefix" default=""/>
-<link name="$(arg tf_prefix)base_link">
+<link name="$(arg tf_prefix)/base_link">
   <inertial>
     <origin rpy="0 0 0" xyz="-0.006946610886831786 0.0035780166273227205 -0.0003164257368845329"/>
@@ -27,5 +27,5 @@
   </collision>
 </link>
-<link name="$(arg tf_prefix)motor_1">
+<link name="$(arg tf_prefix)/motor_1">
   <inertial>
     <origin rpy="0 0 0" xyz="-0.010000306616649128 3.469446951953614e-18 1.4668454062330035e-17"/>
@@ -49,5 +49,5 @@
   </collision>
 </link>
-<link name="$(arg tf_prefix)finger_1">
+<link name="$(arg tf_prefix)/finger_1">
   <inertial>
     <origin rpy="0 0 0" xyz="0.0008908942564820792 0.0264560567515969 0.005010079496025799"/>
@@ -71,5 +71,5 @@
   </collision>
 </link>
-<link name="$(arg tf_prefix)finger_2">
+<link name="$(arg tf_prefix)/finger_2">
   <inertial>
     <origin rpy="0 0 0" xyz="-0.0008915074897803414 0.0264560567515969 -0.005010079496025876"/>
@@ -95,11 +95,11 @@
 <joint name="Rigid1" type="fixed">
   <origin rpy="0 0 0" xyz="-0.057167 0.016 0.0"/>
-  <parent link="$(arg tf_prefix)base_link"/>
-  <child link="$(arg tf_prefix)motor_1"/>
+  <parent link="$(arg tf_prefix)/base_link"/>
+  <child link="$(arg tf_prefix)/motor_1"/>
 </joint>
 <joint name="Slider2" type="prismatic">
   <origin rpy="0 0 0" xyz="-0.005667 0.016 0.0"/>
-  <parent link="$(arg tf_prefix)base_link"/>
-  <child link="$(arg tf_prefix)finger_1"/>
+  <parent link="$(arg tf_prefix)/base_link"/>
+  <child link="$(arg tf_prefix)/finger_1"/>
   <axis xyz="1.0 0.0 -0.0"/>
   <limit effort="100" lower="-0.035" upper="0.0025" velocity="100"/>
@@ -107,6 +107,6 @@
 <joint name="Slider3" type="prismatic">
   <origin rpy="0 0 0" xyz="0.003833 0.016 0.0"/>
-  <parent link="$(arg tf_prefix)base_link"/>
-  <child link="$(arg tf_prefix)finger_2"/>
+  <parent link="$(arg tf_prefix)/base_link"/>
+  <child link="$(arg tf_prefix)/finger_2"/>
   <axis xyz="1.0 0.0 -0.0"/>
   <limit effort="100" lower="0.0" upper="0.0" velocity="100"/>
