Commit message: free -> o

File: obot_urdf_description/urdf/materials.xacro (robot description, xacro)
@@ -1,4 +1,4 @@
 <?xml version="1.0" ?>
-<robot name="freebot_urdf" xmlns:xacro="http://www.ros.org/wiki/xacro" >
+<robot name="obot_urdf" xmlns:xacro="http://www.ros.org/wiki/xacro" >
 <material name="Aluminum - Anodized Rough (Grey)">
   <color rgba="0.5372549019607843 0.5372549019607843 0.5372549019607843 1.0"/>

File: obot_urdf_description/urdf/obot_urdf.urdf (robot description, URDF)
Before this commit: robot freebot_urdf, 10 links, 9 joints
Links:
- link /OS_Connector_Elbow_07b_1: geometry collision mesh filename=package://obot_urdf_description/meshes/OS_Connector_Elbow_0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 scale=0.001 0.001 0.001; visual mesh filename=package://obot_urdf_description/meshes/OS_Connector_Elbow_0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 scale=0.001 0.001 0.001
- link /OS_Connector_Elbow_07e_1: geometry collision mesh filename=package://obot_urdf_description/meshes/OS_Connector_Elbow_0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 scale=0.001 0.001 0.001; visual mesh filename=package://obot_urdf_description/meshes/OS_Connector_Elbow_0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 scale=0.001 0.001 0.001
- link /OS_Connector_shoulder_08_1: geometry collision mesh filename=package://obot_urdf_description/meshes/OS_Connector_shoulde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 scale=0.001 0.001 0.001; visual mesh filename=package://obot_urdf_description/meshes/OS_Connector_shoulde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 scale=0.001 0.001 0.001
- link /OS_Shoulder_connector_01d_1: geometry collision mesh filename=package://obot_urdf_description/meshes/OS_Shoulder_connecto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 scale=0.001 0.001 0.001; visual mesh filename=package://obot_urdf_description/meshes/OS_Shoulder_connecto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 scale=0.001 0.001 0.001
- link /OS_Shoulder_connector_06c_1: geometry collision mesh filename=package://obot_urdf_description/meshes/OS_Shoulder_connecto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 scale=0.001 0.001 0.001; visual mesh filename=package://obot_urdf_description/meshes/OS_Shoulder_connecto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 scale=0.001 0.001 0.001
- link /OS_Tool_Adapter_1: geometry collision mesh filename=package://obot_urdf_description/meshes/OS_Tool_Adapter_1.stl scale=0.001 0.001 0.001; visual mesh filename=package://obot_urdf_description/meshes/OS_Tool_Adapter_1_ob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 scale=0.001 0.001 0.001
- link /OS_Upper_arm_tube_1: geometry collision mesh filename=package://obot_urdf_description/meshes/OS_Upper_arm_tube_1.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 scale=0.001 0.001 0.001; visual mesh filename=package://obot_urdf_description/meshes/OS_Upper_arm_tube_1_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 scale=0.001 0.001 0.001
- link /OS_Upper_arm_tube_2: geometry collision mesh filename=package://obot_urdf_description/meshes/OS_Upper_arm_tube_2.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 scale=0.001 0.001 0.001; visual mesh filename=package://obot_urdf_description/meshes/OS_Upper_arm_tube_2_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 scale=0.001 0.001 0.001
- link /OS_Wrist_connector_01_1: geometry collision mesh filename=package://obot_urdf_description/meshes/OS_Wrist_connector_0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 scale=0.001 0.001 0.001; visual mesh filename=package://obot_urdf_description/meshes/OS_Wrist_connector_0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 scale=0.001 0.001 0.001
- link /base_link: geometry collision mesh filename=package://obot_urdf_description/meshes/base_link.stl scale=0.001 0.001 0.001; visual mesh filename=package://obot_urdf_description/meshes/base_link_obot_urdf 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 scale=0.001 0.001 0.001

File: obot_urdf_description/urdf/obot_urdf.xacro (robot description, xacro)
@@ -1,8 +1,8 @@
 <?xml version="1.0" ?>
-<robot name="freebot_urdf" xmlns:xacro="http://www.ros.org/wiki/xacro">
+<robot name="obot_urdf" xmlns:xacro="http://www.ros.org/wiki/xacro">
 <xacro:arg name="tf_prefix" default=""/>
-<xacro:include filename="$(find freebot_urdf_description)/urdf/materials.xacro" />
-<xacro:include filename="$(find freebot_urdf_description)/urdf/freebot_urdf.trans" />
-<xacro:include filename="$(find freebot_urdf_description)/urdf/freebot_urdf.gazebo" />
+<xacro:include filename="$(find obot_urdf_description)/urdf/materials.xacro" />
+<xacro:include filename="$(find obot_urdf_description)/urdf/obot_urdf.trans" />
+<xacro:include filename="$(find obot_urdf_description)/urdf/obot_urdf.gazebo" />
 <link name="$(arg tf_prefix)/base_link">
   <inertial>
@@ -14,5 +14,5 @@
     <origin rpy="0 0 0" xyz="0 0 0"/>
     <geometry>
-      <mesh filename="package://freebot_urdf_description/meshes/base_link_freebot_urdf v0_Body1_base_link.stl" scale="0.001 0.001 0.001"/>
+      <mesh filename="package://obot_urdf_description/meshes/base_link_obot_urdf v0_Body1_base_link.stl" scale="0.001 0.001 0.001"/>
     </geometry>
     <material name="black">
@@ -23,5 +23,5 @@
     <origin rpy="0 0 0" xyz="0 0 0"/>
     <geometry>
-      <mesh filename="package://freebot_urdf_description/meshes/base_link_freebot_urdf v0_Body2_base_link.stl" scale="0.001 0.001 0.001"/>
+      <mesh filename="package://obot_urdf_description/meshes/base_link_obot_urdf v0_Body2_base_link.stl" scale="0.001 0.001 0.001"/>
     </geometry>
     <material name="black">
@@ -32,5 +32,5 @@
     <origin rpy="0 0 0" xyz="0 0 0"/>
     <geometry>
-      <mesh filename="package://freebot_urdf_description/meshes/base_link.stl" scale="0.001 0.001 0.001"/>
+      <mesh filename="package://obot_urdf_description/meshes/base_link.stl" scale="0.001 0.001 0.001"/>
     </geometry>
   </collision>
@@ -45,5 +45,5 @@
     <origin rpy="0 0 0" xyz="0.006 0.0 -0.1215"/>
     <geometry>
-      <mesh filename="package://freebot_urdf_description/meshes/OS_Shoulder_connector_06c_1_freebot_urdf v0_Body1_OS_Shoulder_connector_06c_1.stl" scale="0.001 0.001 0.001"/>
+      <mesh filename="package://obot_urdf_description/meshes/OS_Shoulder_connector_06c_1_obot_urdf v0_Body1_OS_Shoulder_connector_06c_1.stl" scale="0.001 0.001 0.001"/>
     </geometry>
     <material name="black">
@@ -54,5 +54,5 @@
     <origin rpy="0 0 0" xyz="0.006 0.0 -0.1215"/>
     <geometry>
-      <mesh filename="package://freebot_urdf_description/meshes/OS_Shoulder_connector_06c_1_freebot_urdf v0_Body2_OS_Shoulder_connector_06c_1.stl" scale="0.001 0.001 0.001"/>
+      <mesh filename="package://obot_urdf_description/meshes/OS_Shoulder_connector_06c_1_obot_urdf v0_Body2_OS_Shoulder_connector_06c_1.stl" scale="0.001 0.001 0.001"/>
     </geometry>
     <material name="blue1">
@@ -63,5 +63,5 @@
     <origin rpy="0 0 0" xyz="0.006 0.0 -0.1215"/>
     <geometry>
-      <mesh filename="package://freebot_urdf_description/meshes/OS_Shoulder_connector_06c_1.stl" scale="0.001 0.001 0.001"/>
+      <mesh filename="package://obot_urdf_description/meshes/OS_Shoulder_connector_06c_1.stl" scale="0.001 0.001 0.001"/>
     </geometry>
   </collision>
@@ -76,5 +76,5 @@
     <origin rpy="0 0 0" xyz="0.0035 0.0 -0.4215"/>
     <geometry>
-      <mesh filename="package://freebot_urdf_description/meshes/OS_Connector_shoulder_08_1_freebot_urdf v0_Body1_OS_Connector_shoulder_08_1.stl" scale="0.001 0.001 0.001"/>
+      <mesh filename="package://obot_urdf_description/meshes/OS_Connector_shoulder_08_1_obot_urdf v0_Body1_OS_Connector_shoulder_08_1.stl" scale="0.001 0.001 0.001"/>
     </geometry>
     <material name="black">
@@ -85,5 +85,5 @@
     <origin rpy="0 0 0" xyz="0.0035 0.0 -0.4215"/>
     <geometry>
-      <mesh filename="package://freebot_urdf_description/meshes/OS_Connector_shoulder_08_1_freebot_urdf v0_Body2_OS_Connector_shoulder_08_1.stl" scale="0.001 0.001 0.001"/>
+      <mesh filename="package://obot_urdf_description/meshes/OS_Connector_shoulder_08_1_obot_urdf v0_Body2_OS_Connector_shoulder_08_1.stl" scale="0.001 0.001 0.001"/>
     </geometry>
     <material name="blue2">
@@ -94,5 +94,5 @@
     <origin rpy="0 0 0" xyz="0.0035 0.0 -0.4215"/>
     <geometry>
-      <mesh filename="package://freebot_urdf_description/meshes/OS_Connector_shoulder_08_1.stl" scale="0.001 0.001 0.001"/>
+      <mesh filename="package://obot_urdf_description/meshes/OS_Connector_shoulder_08_1.stl" scale="0.001 0.001 0.001"/>
     </geometry>
   </collision>
@@ -107,5 +107,5 @@
     <origin rpy="0 0 0" xyz="-0.0583 0.3 -0.4215"/>
     <geometry>
-      <mesh filename="package://freebot_urdf_description/meshes/OS_Wrist_connector_01_1_freebot_urdf v0_Body1_OS_Wrist_connector_01_1.stl" scale="0.001 0.001 0.001"/>
+      <mesh filename="package://obot_urdf_description/meshes/OS_Wrist_connector_01_1_obot_urdf v0_Body1_OS_Wrist_connector_01_1.stl" scale="0.001 0.001 0.001"/>
     </geometry>
     <material name="black">
@@ -116,5 +116,5 @@
     <origin rpy="0 0 0" xyz="-0.0583 0.3 -0.4215"/>
     <geometry>
-      <mesh filename="package://freebot_urdf_description/meshes/OS_Wrist_connector_01_1_freebot_urdf v0_Body2_OS_Wrist_connector_01_1.stl" scale="0.001 0.001 0.001"/>
+      <mesh filename="package://obot_urdf_description/meshes/OS_Wrist_connector_01_1_obot_urdf v0_Body2_OS_Wrist_connector_01_1.stl" scale="0.001 0.001 0.001"/>
     </geometry>
     <material name="blue1">
@@ -125,5 +125,5 @@
     <origin rpy="0 0 0" xyz="-0.0583 0.3 -0.4215"/>
     <geometry>
-      <mesh filename="package://freebot_urdf_description/meshes/OS_Wrist_connector_01_1.stl" scale="0.001 0.001 0.001"/>
+      <mesh filename="package://obot_urdf_description/meshes/OS_Wrist_connector_01_1.stl" scale="0.001 0.001 0.001"/>
     </geometry>
   </collision>
@@ -138,5 +138,5 @@
     <origin rpy="0 0 0" xyz="0.0 0.0 -0.0605"/>
     <geometry>
-      <mesh filename="package://freebot_urdf_description/meshes/OS_Shoulder_connector_01d_1_freebot_urdf v0_Body1_OS_Shoulder_connector_01d_1.stl" scale="0.001 0.001 0.001"/>
+      <mesh filename="package://obot_urdf_description/meshes/OS_Shoulder_connector_01d_1_obot_urdf v0_Body1_OS_Shoulder_connector_01d_1.stl" scale="0.001 0.001 0.001"/>
     </geometry>
     <material name="blue1">
@@ -147,5 +147,5 @@
     <origin rpy="0 0 0" xyz="0.0 0.0 -0.0605"/>
     <geometry>
-      <mesh filename="package://freebot_urdf_description/meshes/OS_Shoulder_connector_01d_1_freebot_urdf v0_Body2_OS_Shoulder_connector_01d_1.stl" scale="0.001 0.001 0.001"/>
+      <mesh filename="package://obot_urdf_description/meshes/OS_Shoulder_connector_01d_1_obot_urdf v0_Body2_OS_Shoulder_connector_01d_1.stl" scale="0.001 0.001 0.001"/>
     </geometry>
     <material name="black">
@@ -156,5 +156,5 @@
     <origin rpy="0 0 0" xyz="0.0 0.0 -0.0605"/>
     <geometry>
-      <mesh filename="package://freebot_urdf_description/meshes/OS_Shoulder_connector_01d_1.stl" scale="0.001 0.001 0.001"/>
+      <mesh filename="package://obot_urdf_description/meshes/OS_Shoulder_connector_01d_1.stl" scale="0.001 0.001 0.001"/>
     </geometry>
   </collision>
@@ -169,5 +169,5 @@
     <origin rpy="0 0 0" xyz="-0.0943 0.3385 -0.4215"/>
     <geometry>
-      <mesh filename="package://freebot_urdf_description/meshes/OS_Tool_Adapter_1_freebot_urdf v0_Body1_OS_Tool_Adapter_1.stl" scale="0.001 0.001 0.001"/>
+      <mesh filename="package://obot_urdf_description/meshes/OS_Tool_Adapter_1_obot_urdf v0_Body1_OS_Tool_Adapter_1.stl" scale="0.001 0.001 0.001"/>
     </geometry>
     <material name="aluminum">
@@ -178,5 +178,5 @@
     <origin rpy="0 0 0" xyz="-0.0943 0.3385 -0.4215"/>
     <geometry>
-      <mesh filename="package://freebot_urdf_description/meshes/OS_Tool_Adapter_1.stl" scale="0.001 0.001 0.001"/>
+      <mesh filename="package://obot_urdf_description/meshes/OS_Tool_Adapter_1.stl" scale="0.001 0.001 0.001"/>
     </geometry>
   </collision>
@@ -191,5 +191,5 @@
     <origin rpy="0 0 0" xyz="0.0344 0.0 -0.1635"/>
     <geometry>
-      <mesh filename="package://freebot_urdf_description/meshes/OS_Upper_arm_tube_1_freebot_urdf v0_Body1_OS_Upper_arm_tube_1.stl" scale="0.001 0.001 0.001"/>
+      <mesh filename="package://obot_urdf_description/meshes/OS_Upper_arm_tube_1_obot_urdf v0_Body1_OS_Upper_arm_tube_1.stl" scale="0.001 0.001 0.001"/>
     </geometry>
     <material name="aluminum">
@@ -200,5 +200,5 @@
     <origin rpy="0 0 0" xyz="0.0344 0.0 -0.1635"/>
     <geometry>
-      <mesh filename="package://freebot_urdf_description/meshes/OS_Upper_arm_tube_1.stl" scale="0.001 0.001 0.001"/>
+      <mesh filename="package://obot_urdf_description/meshes/OS_Upper_arm_tube_1.stl" scale="0.001 0.001 0.001"/>
     </geometry>
   </collision>
@@ -213,5 +213,5 @@
     <origin rpy="0 0 0" xyz="0.0344 0.0 -0.3845"/>
     <geometry>
-      <mesh filename="package://freebot_urdf_description/meshes/OS_Connector_Elbow_07b_1_freebot_urdf v0_Body1_OS_Connector_Elbow_07b_1.stl" scale="0.001 0.001 0.001"/>
+      <mesh filename="package://obot_urdf_description/meshes/OS_Connector_Elbow_07b_1_obot_urdf v0_Body1_OS_Connector_Elbow_07b_1.stl" scale="0.001 0.001 0.001"/>
     </geometry>
     <material name="black">
@@ -222,5 +222,5 @@
     <origin rpy="0 0 0" xyz="0.0344 0.0 -0.3845"/>
     <geometry>
-      <mesh filename="package://freebot_urdf_description/meshes/OS_Connector_Elbow_07b_1_freebot_urdf v0_Body2_OS_Connector_Elbow_07b_1.stl" scale="0.001 0.001 0.001"/>
+      <mesh filename="package://obot_urdf_description/meshes/OS_Connector_Elbow_07b_1_obot_urdf v0_Body2_OS_Connector_Elbow_07b_1.stl" scale="0.001 0.001 0.001"/>
     </geometry>
     <material name="blue1">
@@ -231,5 +231,5 @@
     <origin rpy="0 0 0" xyz="0.0344 0.0 -0.3845"/>
     <geometry>
-      <mesh filename="package://freebot_urdf_description/meshes/OS_Connector_Elbow_07b_1.stl" scale="0.001 0.001 0.001"/>
+      <mesh filename="package://obot_urdf_description/meshes/OS_Connector_Elbow_07b_1.stl" scale="0.001 0.001 0.001"/>
     </geometry>
   </collision>
@@ -244,5 +244,5 @@
     <origin rpy="0 0 0" xyz="-0.0274 0.038 -0.4215"/>
     <geometry>
-      <mesh filename="package://freebot_urdf_description/meshes/OS_Upper_arm_tube_2_freebot_urdf v0_Body1_OS_Upper_arm_tube_2.stl" scale="0.001 0.001 0.001"/>
+      <mesh filename="package://obot_urdf_description/meshes/OS_Upper_arm_tube_2_obot_urdf v0_Body1_OS_Upper_arm_tube_2.stl" scale="0.001 0.001 0.001"/>
     </geometry>
     <material name="aluminum">
@@ -253,5 +253,5 @@
     <origin rpy="0 0 0" xyz="-0.0274 0.038 -0.4215"/>
     <geometry>
-      <mesh filename="package://freebot_urdf_description/meshes/OS_Upper_arm_tube_2.stl" scale="0.001 0.001 0.001"/>
+      <mesh filename="package://obot_urdf_description/meshes/OS_Upper_arm_tube_2.stl" scale="0.001 0.001 0.001"/>
     </geometry>
   </collision>
@@ -266,5 +266,5 @@
     <origin rpy="0 0 0" xyz="-0.0274 0.259 -0.4215"/>
     <geometry>
-      <mesh filename="package://freebot_urdf_description/meshes/OS_Connector_Elbow_07e_1_freebot_urdf v0_Body1_OS_Connector_Elbow_07e_1.stl" scale="0.001 0.001 0.001"/>
+      <mesh filename="package://obot_urdf_description/meshes/OS_Connector_Elbow_07e_1_obot_urdf v0_Body1_OS_Connector_Elbow_07e_1.stl" scale="0.001 0.001 0.001"/>
     </geometry>
     <material name="black">
@@ -275,5 +275,5 @@
     <origin rpy="0 0 0" xyz="-0.0274 0.259 -0.4215"/>
     <geometry>
-      <mesh filename="package://freebot_urdf_description/meshes/OS_Connector_Elbow_07e_1_freebot_urdf v0_Body2_OS_Connector_Elbow_07e_1.stl" scale="0.001 0.001 0.001"/>
+      <mesh filename="package://obot_urdf_description/meshes/OS_Connector_Elbow_07e_1_obot_urdf v0_Body2_OS_Connector_Elbow_07e_1.stl" scale="0.001 0.001 0.001"/>
     </geometry>
     <material name="blue1">
@@ -284,5 +284,5 @@
     <origin rpy="0 0 0" xyz="-0.0274 0.259 -0.4215"/>
     <geometry>
-      <mesh filename="package://freebot_urdf_description/meshes/OS_Connector_Elbow_07e_1.stl" scale="0.001 0.001 0.001"/>
+      <mesh filename="package://obot_urdf_description/meshes/OS_Connector_Elbow_07e_1.stl" scale="0.001 0.001 0.001"/>
     </geometry>
   </collision>
